Commit message: organize, photos, remove phantomx_descrition dependence

File: urdf/phantomx.urdf (robot description, URDF)
Before this commit: robot PhantomX, 26 links, 25 joints
Links:
- link MP_BODY: geometry collision mesh filename=package://phantomx_ros/meshes/body_coll.STL scale=1 1 1; visual mesh filename=package://phantomx_ros/meshes/body.STL scale=1 1 1
- link c1_lf: geometry collision mesh filename=package://phantomx_ros/meshes/connect_coll.STL scale=1 1 1; visual mesh filename=package://phantomx_ros/meshes/connect.STL scale=1 1 1
- link c1_lm: geometry collision mesh filename=package://phantomx_ros/meshes/connect_coll.STL scale=1 1 1; visual mesh filename=package://phantomx_ros/meshes/connect.STL scale=1 1 1
- link c1_lr: geometry collision mesh filename=package://phantomx_ros/meshes/connect_coll.STL scale=1 1 1; visual mesh filename=package://phantomx_ros/meshes/connect.STL scale=1 1 1
- link c1_rf: geometry collision mesh filename=package://phantomx_ros/meshes/connect_coll.STL scale=1 1 1; visual mesh filename=package://phantomx_ros/meshes/connect.STL scale=1 1 1
- link c1_rm: geometry collision mesh filename=package://phantomx_ros/meshes/connect_coll.STL scale=1 1 1; visual mesh filename=package://phantomx_ros/meshes/connect.STL scale=1 1 1
- link c1_rr: geometry collision mesh filename=package://phantomx_ros/meshes/connect_coll.STL scale=1 1 1; visual mesh filename=package://phantomx_ros/meshes/connect.STL scale=1 1 1
- link c2_lf: geometry collision mesh filename=package://phantomx_ros/meshes/connect_coll.STL scale=1 1 1; visual mesh filename=package://phantomx_ros/meshes/connect.STL scale=1 1 1
- link c2_lm: geometry collision mesh filename=package://phantomx_ros/meshes/connect_coll.STL scale=1 1 1; visual mesh filename=package://phantomx_ros/meshes/connect.STL scale=1 1 1
- link c2_lr: geometry collision mesh filename=package://phantomx_ros/meshes/connect_coll.STL scale=1 1 1; visual mesh filename=package://phantomx_ros/meshes/connect.STL scale=1 1 1
- link c2_rf: geometry collision mesh filename=package://phantomx_ros/meshes/connect_coll.STL scale=1 1 1; visual mesh filename=package://phantomx_ros/meshes/connect.STL scale=1 1 1
- link c2_rm: geometry collision mesh filename=package://phantomx_ros/meshes/connect_coll.STL scale=1 1 1; visual mesh filename=package://phantomx_ros/meshes/connect.STL scale=1 1 1
- link c2_rr: geometry collision mesh filename=package://phantomx_ros/meshes/connect_coll.STL scale=1 1 1; visual mesh filename=package://phantomx_ros/meshes/connect.STL scale=1 1 1
- link thigh_lf: geometry collision mesh filename=package://phantomx_ros/meshes/thigh_l_coll.STL scale=1 1 1; visual mesh filename=package://phantomx_ros/meshes/thigh_l.STL scale=1 1 1
- link thigh_lm: geometry collision mesh filename=package://phantomx_ros/meshes/thigh_l_coll.STL scale=1 1 1; visual mesh filename=package://phantomx_ros/meshes/thigh_l.STL scale=1 1 1
- link thigh_lr: geometry collision mesh filename=package://phantomx_ros/meshes/thigh_l_coll.STL scale=1 1 1; visual mesh filename=package://phantomx_ros/meshes/thigh_l.STL scale=1 1 1
- link thigh_rf: geometry collision mesh filename=package://phantomx_ros/meshes/thigh_l_coll.STL scale=1 1 1; visual mesh filename=package://phantomx_ros/meshes/thigh_l.STL scale=1 1 1
- link thigh_rm: geometry collision mesh filename=package://phantomx_ros/meshes/thigh_l_coll.STL scale=1 1 1; visual mesh filename=package://phantomx_ros/meshes/thigh_l.STL scale=1 1 1
- link thigh_rr: geometry collision mesh filename=package://phantomx_ros/meshes/thigh_l_coll.STL scale=1 1 1; visual mesh filename=package://phantomx_ros/meshes/thigh_l.STL scale=1 1 1
- link tibia_lf: geometry collision mesh filename=package://phantomx_ros/meshes/tibia_l_coll.STL scale=1 1 1; visual mesh filename=package://phantomx_ros/meshes/tibia_l.STL scale=1 1 1
- link tibia_lm: geometry collision mesh filename=package://phantomx_ros/meshes/tibia_l_coll.STL scale=1 1 1; visual mesh filename=package://phantomx_ros/meshes/tibia_l.STL scale=1 1 1
- link tibia_lr: geometry collision mesh filename=package://phantomx_ros/meshes/tibia_l_coll.STL scale=1 1 1; visual mesh filename=package://phantomx_ros/meshes/tibia_l.STL scale=1 1 1
- link tibia_rf: geometry collision mesh filename=package://phantomx_ros/meshes/tibia_l_coll.STL scale=1 1 1; visual mesh filename=package://phantomx_ros/meshes/tibia_l.STL scale=1 1 1
- link tibia_rm: geometry collision mesh filename=package://phantomx_ros/meshes/tibia_l_coll.STL scale=1 1 1; visual mesh filename=package://phantomx_ros/meshes/tibia_l.STL scale=1 1 1
- link tibia_rr: geometry collision mesh filename=package://phantomx_ros/meshes/tibia_l_coll.STL scale=1 1 1; visual mesh filename=package://phantomx_ros/meshes/tibia_l.STL scale=1 1 1
